File: teensy-sdr.kicad_pcb (KiCad board)
At the start: 2 copper layers, 102 x 76.5 mm, 63 parts, among them J1 Conn_Coaxial, J2 Battery, J3 AudioJack3_SwitchT, J4 USB_C_Receptacle_USB2.0_16P, SW1 MSK-12C02 SPDT, U1 Teensy4.0, U2 Si4735-D60-GU, U3 AS179-92LF, U4 SN74LVC1G14DBV, U5 TPS63030DSK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

Commit message: PCB Refractor
Parts:
- L1: value L -> 1.5uF; footprint Inductor_SMD:L_10.4x10.4_H4.8 -> Inductor_SMD:L_7.3x7.3_H3.5
- R1: value 600R -> 1k
- moved J2 40.7 mm to (190.8, 133.1)
- moved SW1 32.0 mm to (195.3, 122.3)
- moved U1 29.8 mm to (146.1, 124.5)
- moved U6 28.3 mm to (184.4, 113.7)
- moved R15 27.8 mm to (179.5, 112.0)
- moved R13 26.3 mm to (183.5, 107.5), turned to -90 degrees
- moved R22 25.3 mm to (191.2, 119.0), turned to -90 degrees
- moved R14 23.8 mm to (185.5, 107.5), turned to -90 degrees
- moved C10 20.5 mm to (159.2, 98.7)
- moved C3 20.5 mm to (145.2, 98.7)
- moved C5 20.5 mm to (136.2, 99.7)
- moved C6 20.5 mm to (139.2, 99.7)
- moved C7 20.5 mm to (155.2, 94.7)
- moved C8 20.5 mm to (156.8, 98.8)
- moved R10 20.5 mm to (146.8, 95.7)
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Connections:
- R13 pad 1: Net-(SW1-A) -> +3V3
- R14 pad 1: Net-(SW1-A) -> +3V3
Routing:
- net AMP_DIN: track 33.2 -> 104.3 mm, vias 0 -> 2
- net AMP_LRCLK: track 17.1 -> 82.7 mm, vias 0 -> 3
- net AMP_BCLK: track 13.9 -> 78.9 mm, vias 0 -> 3
- net SDR_DOUT: track 45.0 -> 93.7 mm, vias 0 -> 2
- net JACK_DETECT: track 29.2 -> 77.1 mm, vias 2 -> 0
- net AMP_CS: track 39.9 -> 85.0 mm, vias 1 -> 2
- net SDR_CS: track 36.0 -> 77.3 mm
- net VIN: track 91.7 -> 54.6 mm
- net AMP_MCLK: track 15.1 -> 50.4 mm, vias 1 -> 2
- net Net-(U1-10_CS_MQSR): track 75.0 -> 109.6 mm
- net OLED_D/C: track 26.0 -> 60.6 mm, vias 0 -> 1
- net OLED_CS: track 29.9 -> 61.9 mm, vias 0 -> 1
- net Net-(U2-DFS): track 34.7 -> 4.48 mm, vias 2 -> 0
- net Net-(SW1-B): track 46.6 -> 17.9 mm
- net Net-(U1-9_OUT1C): track 55.5 -> 82.4 mm, vias 1 -> 2
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