File: teensy-sdr.kicad_pcb (KiCad board)
At the start: 2 copper layers, 102 x 76.5 mm, 63 parts, among them J1 Conn_Coaxial, J2 Battery, J3 AudioJack3_SwitchT, J4 USB_C_Receptacle_USB2.0_16P, SW1 MSK-12C02 SPDT, U1 Teensy4.0, U2 Si4735-D60-GU, U3 AS179-92LF, U4 SN74LVC1G14DBV, U5 TPS63030DSK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

Commit message: fix swapped I2S lines
Connections:
- U1 pad 10: AMP_DIN -> SDR_DOUT
- U1 pad 9: SDR_DOUT -> AMP_DIN
Routing:
- net AMP_DIN: track 104.3 -> 99.4 mm
- net SDR_DOUT: track 93.7 -> 95.0 mm
Changed lines of the file:
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@@
 			(layers "*.Cu" "*.Mask")
 			(remove_unused_layers no)
-			(net 23 "SDR_DOUT")
+			(net 79 "AMP_DIN")
 			(pinfunction "7_RX2_OUT1A")
 			(pintype "bidirectional")
@@
 			(layers "*.Cu" "*.Mask")
 			(remove_unused_layers no)
-			(net 79 "AMP_DIN")
+			(net 23 "SDR_DOUT")
 			(pinfunction "8_TX2_IN1")
 			(pintype "bidirectional")
@@
 	)
 	(segment
-		(start 128.251586 135.253)
-		(end 126.499 133.500414)
+		(start 148.951 135.654)
+		(end 128.085486 135.654)
 		(width 0.2)
 		(layer "F.Cu")
@@
 	)
 	(segment
-		(start 126.284341 109.320131)
-		(end 126.636398 108.968074)
+		(start 126.099 110.198362)
+		(end 125.884341 109.983703)
 		(width 0.2)
 		(layer "F.Cu")
@@
 	)
 	(segment
-		(start 126.499 110.032676)
-		(end 126.284341 109.818017)
+		(start 152.485 132.12)
+		(end 148.951 135.654)
 		(width 0.2)
 		(layer "F.Cu")
@@
 	)
 	(segment
-		(start 142.25 94.485843)
-		(end 142.25 86.85)
+		(start 126.098 117.340686)
+		(end 126.099 117.339686)
 		(width 0.2)
 		(layer "F.Cu")
@@
 	)
 	(segment
-		(start 149.945 132.12)
-		(end 146.812 135.253)
+		(start 125.884341 109.983703)
+		(end 125.884341 109.154446)
 		(width 0.2)
 		(layer "F.Cu")
@@
 	)
 	(segment
-		(start 146.812 135.253)
-		(end 128.251586 135.253)
+		(start 126.099 117.339686)
+		(end 126.099 110.198362)
 		(width 0.2)
 		(layer "F.Cu")
@@
 	)
 	(segment
-		(start 126.284341 109.818017)
-		(end 126.284341 109.320131)
+		(start 127.301384 108.568074)
+		(end 127.451027 108.717717)
 		(width 0.2)
 		(layer "F.Cu")
@@
 	)
 	(segment
-		(start 127.134284 108.968074)
-		(end 127.451027 109.284817)
+		(start 125.884341 109.154446)
+		(end 126.470712 108.568074)
 		(width 0.2)
 		(layer "F.Cu")
@@
 	)
 	(segment
-		(start 126.499 133.500414)
-		(end 126.499 110.032676)
+		(start 139.75 96.418743)
+		(end 139.75 86.85)
 		(width 0.2)
 		(layer "F.Cu")
@@
 	)
 	(segment
-		(start 127.451027 109.284817)
-		(end 142.25 94.485843)
+		(start 127.451027 108.717717)
+		(end 139.75 96.418743)
 		(width 0.2)
 		(layer "F.Cu")
@@
 	)
 	(segment
-		(start 126.636398 108.968074)
-		(end 127.134284 108.968074)
+		(start 126.470712 108.568074)
+		(end 127.301384 108.568074)
+		(width 0.2)
+		(layer "F.Cu")
+		(net 23)
+	)
+	(segment
+		(start 126.098 133.666514)
+		(end 126.098 117.340686)
+		(width 0.2)
+		(layer "F.Cu")
+		(net 23)
+	)
+	(segment
+		(start 128.085486 135.654)
+		(end 126.098 133.666514)
 		(width 0.2)
 		(layer "F.Cu")
@@
 	)
 	(via
-		(at 142.25 86.85)
+		(at 139.75 86.85)
 		(size 0.6)
 		(drill 0.3)
@@
 	)
 	(segment
-		(start 137.75 74.75)
-		(end 142.25 79.25)
+		(start 139.75 86.85)
+		(end 139.75 76.75)
 		(width 0.2)
 		(layer "B.Cu")
@@
 	)
 	(segment
-		(start 142.25 79.25)
-		(end 142.25 86.85)
+		(start 139.75 76.75)
+		(end 137.75 74.75)
 		(width 0.2)
 		(layer "B.Cu")
@@
 	)
 	(segment
-		(start 148.951 135.654)
-		(end 128.085486 135.654)
+		(start 128.251586 135.253)
+		(end 126.499 133.500414)
 		(width 0.2)
 		(layer "F.Cu")
@@
 	)
 	(segment
-		(start 126.099 110.198362)
-		(end 125.884341 109.983703)
+		(start 126.284341 109.320131)
+		(end 126.636398 108.968074)
 		(width 0.2)
 		(layer "F.Cu")
@@
 	)
 	(segment
-		(start 152.485 132.12)
-		(end 148.951 135.654)
+		(start 126.499 110.032676)
+		(end 126.284341 109.818017)
 		(width 0.2)
 		(layer "F.Cu")
@@
 	)
 	(segment
-		(start 148.149999 78.25)
-		(end 139.75 78.25)
+		(start 151.275 74.3875)
+		(end 151.275 75.124999)
 		(width 0.2)
 		(layer "F.Cu")
@@
 	)
 	(segment
-		(start 126.098 117.340686)
-		(end 126.099 117.339686)
+		(start 142.25 94.485843)
+		(end 142.25 86.85)
 		(width 0.2)
 		(layer "F.Cu")
@@
 	)
 	(segment
-		(start 125.884341 109.983703)
-		(end 125.884341 109.154446)
+		(start 149.945 132.12)
+		(end 146.812 135.253)
 		(width 0.2)
 		(layer "F.Cu")
@@
 	)
 	(segment
-		(start 126.099 117.339686)
-		(end 126.099 110.198362)
+		(start 146.812 135.253)
+		(end 128.251586 135.253)
 		(width 0.2)
 		(layer "F.Cu")
@@
 	)
 	(segment
-		(start 127.301384 108.568074)
-		(end 127.451027 108.717717)
-		(width 0.2)
-		(layer "F.Cu")
-		(net 79)
-	)
-	(segment
-		(start 151.275 74.3875)
-		(end 151.275 75.124999)
-		(width 0.2)
-		(layer "F.Cu")
-		(net 79)
-	)
-	(segment
-		(start 125.884341 109.154446)
-		(end 126.470712 108.568074)
+		(start 126.284341 109.818017)
+		(end 126.284341 109.320131)
 		(width 0.2)
 		(layer "F.Cu")
@@
 	)
 	(segment
-		(start 139.75 96.418743)
-		(end 139.75 86.85)
+		(start 127.134284 108.968074)
+		(end 127.451027 109.284817)
 		(width 0.2)
 		(layer "F.Cu")
@@
 	)
 	(segment
-		(start 127.451027 108.717717)
-		(end 139.75 96.418743)
+		(start 126.499 133.500414)
+		(end 126.499 110.032676)
 		(width 0.2)
 		(layer "F.Cu")
@@
 	)
 	(segment
-		(start 126.470712 108.568074)
-		(end 127.301384 108.568074)
+		(start 148.149999 78.25)
+		(end 142.25 78.25)
 		(width 0.2)
 		(layer "F.Cu")
@@
 	)
 	(segment
-		(start 126.098 133.666514)
-		(end 126.098 117.340686)
+		(start 127.451027 109.284817)
+		(end 142.25 94.485843)
 		(width 0.2)
 		(layer "F.Cu")
@@
 	)
 	(segment
-		(start 128.085486 135.654)
-		(end 126.098 133.666514)
+		(start 126.636398 108.968074)
+		(end 127.134284 108.968074)
 		(width 0.2)
 		(layer "F.Cu")
@@
 	)
 	(via
-		(at 139.75 86.85)
+		(at 142.25 86.85)
 		(size 0.6)
 		(drill 0.3)
@@
 	)
 	(via
-		(at 139.75 78.25)
+		(at 142.25 78.25)
 		(size 0.6)
 		(drill 0.3)
@@
 	)
 	(segment
-		(start 139.75 86.85)
-		(end 139.75 78.25)
+		(start 142.25 78.25)
+		(end 142.25 86.85)
 		(width 0.2)
 		(layer "B.Cu")
